File: LEDregulator.sch (KiCad schematic (older format))
At the start: 28 parts, among them J1 2.1mm DC jack, J2 2way Screw Terminal, J3 2way Screw Terminal, SW1 DPDT Switch, SW2 6pos rotary

Commit message: Added first board components
Parts:
- C1: footprint (none) -> Capacitors_SMD:C_1206
- C2: footprint (none) -> Capacitors_SMD:CP_Elec_8x10.5
- C3, C4: footprint (none) -> Capacitors_SMD:C_0603
- DC1: symbol jakub:LDU2430S1000 -> LEDregulator-rescue:LDU2430S1000-jakub
- J1: footprint (none) -> jakub:2.1mmBarrelJack
- J2, J3: footprint (none) -> Terminal_Blocks:TerminalBlock_bornier-2_P5.08mm
- R1, R10, R11, R12, R13, R14, R15, R16, R2, R3, R4, R5, R6, R7, R8, R9: footprint (none) -> Resistors_SMD:R_0603
- SW2: symbol jakub:SW_Rotary1x6 -> LEDregulator-rescue:SW_Rotary1x6-jakub
Changed lines of the file:
@@
 $EndDescr
 $Comp
-L jakub:SW_Rotary1x6 SW2
+L LEDregulator-rescue:SW_Rotary1x6-jakub SW2
 U 1 1 5CE493DC
 P 5700 4150
@@
 F 0 "J1" H 1355 1917 50  0000 C CNN
 F 1 "2.1mm DC jack" H 1355 1826 50  0000 C CNN
-F 2 "" H 1350 1560 50  0001 C CNN
+F 2 "jakub:2.1mmBarrelJack" H 1350 1560 50  0001 C CNN
 F 3 "~" H 1350 1560 50  0001 C CNN
 F 4 "FC681478" H 1300 1600 50  0001 C CNN "Part Number"
-F 5 "Farnell" H 1300 1600 50  0001 C CNN "Distributor"
-F 6 "Cliff Electronics" H 1300 1600 50  0001 C CNN "Manufacturer"
-F 7 "2450496" H 1300 1600 50  0001 C CNN "Order Code"
+F 5 "Cliff Electronics" H 1300 1600 50  0001 C CNN "Manufacturer"
+F 6 "2450496" H 1300 1600 50  0001 C CNN "Order Code"
+F 7 "Farnell" H 1300 1600 50  0001 C CNN "Distributor"
 F 8 "2.1mm 2A/16V DC power jack" H 1300 1600 50  0001 C CNN "Description"
 	1    1300 1600
@@
 F 0 "R3" V 5550 1100 50  0000 C CNN
 F 1 "150R" V 5650 1100 50  0000 C CNN
-F 2 "" V 5580 1100 50  0001 C CNN
+F 2 "Resistors_SMD:R_0603" V 5580 1100 50  0001 C CNN
 F 3 "~" H 5650 1100 50  0001 C CNN
 F 4 "MCWR06X1500FTL" H 5650 1100 50  0001 C CNN "Part Number"
@@
 F 0 "C2" H 4118 1996 50  0000 L CNN
 F 1 "47u/63V" H 4118 1905 50  0000 L CNN
-F 2 "" H 4038 1800 50  0001 C CNN
+F 2 "Capacitors_SMD:CP_Elec_8x10.5" H 4038 1800 50  0001 C CNN
 F 3 "~" H 4000 1950 50  0001 C CNN
 F 4 "EEE1JA470UP" H 4000 1950 50  0001 C CNN "Part Number"
@@
 F 0 "R10" V 6800 4250 50  0000 C CNN
 F 1 "270R" V 6750 4050 50  0000 C CNN
-F 2 "" V 6680 4050 50  0001 C CNN
+F 2 "Resistors_SMD:R_0603" V 6680 4050 50  0001 C CNN
 F 3 "~" H 6750 4050 50  0001 C CNN
 F 4 "MCWR06X2700FTL" H 6750 4050 50  0001 C CNN "Part Number"
@@
 F 0 "J3" H 8830 1492 50  0000 L CNN
 F 1 "2way Screw Terminal" H 8830 1401 50  0000 L CNN
-F 2 "" H 8750 1500 50  0001 C CNN
+F 2 "Terminal_Blocks:TerminalBlock_bornier-2_P5.08mm" H 8750 1500 50  0001 C CNN
 F 3 "~" H 8750 1500 50  0001 C CNN
 F 4 "CTB0102/2" H 8750 1500 50  0001 C CNN "Part Number"
@@
 F 0 "C3" H 4515 4196 50  0000 L CNN
 F 1 "100n" H 4515 4105 50  0000 L CNN
-F 2 "" H 4438 4000 50  0001 C CNN
+F 2 "Capacitors_SMD:C_0603" H 4438 4000 50  0001 C CNN
 F 3 "~" H 4400 4150 50  0001 C CNN
 F 4 "MC0603B104K500CT" H 4400 4150 50  0001 C CNN "Part Number"
@@
 	5500 1100 2800 1100
 $Comp
-L jakub:LDU2430S1000 DC1
+L LEDregulator-rescue:LDU2430S1000-jakub DC1
 U 1 1 5CE70B4D
 P 5900 1800
@@
 F 0 "C1" H 3315 1996 50  0000 L CNN
 F 1 "10u/50V" H 3315 1905 50  0000 L CNN
-F 2 "" H 3238 1800 50  0001 C CNN
+F 2 "Capacitors_SMD:C_1206" H 3238 1800 50  0001 C CNN
 F 3 "~" H 3200 1950 50  0001 C CNN
 F 4 "GRT31CR61H106KE01L" H 3200 1950 50  0001 C CNN "Part Number"
@@
 F 0 "C4" H 5015 4196 50  0000 L CNN
 F 1 "100n" H 5015 4105 50  0000 L CNN
-F 2 "" H 4938 4000 50  0001 C CNN
+F 2 "Capacitors_SMD:C_0603" H 4938 4000 50  0001 C CNN
 F 3 "~" H 4900 4150 50  0001 C CNN
 F 4 "MC0603B104K500CT" H 4900 4150 50  0001 C CNN "Part Number"
@@
 F 0 "R4" V 6050 1100 50  0000 C CNN
 F 1 "150R" V 6150 1100 50  0000 C CNN
-F 2 "" V 6080 1100 50  0001 C CNN
+F 2 "Resistors_SMD:R_0603" V 6080 1100 50  0001 C CNN
 F 3 "~" H 6150 1100 50  0001 C CNN
 F 4 "MCWR06X1500FTL" H 6150 1100 50  0001 C CNN "Part Number"
@@
 F 0 "R14" V 7200 4050 50  0000 C CNN
 F 1 "150R" V 7250 3850 50  0000 C CNN
-F 2 "" V 7180 3850 50  0001 C CNN
+F 2 "Resistors_SMD:R_0603" V 7180 3850 50  0001 C CNN
 F 3 "~" H 7250 3850 50  0001 C CNN
 F 4 "MCWR06X1500FTL" H 7250 3850 50  0001 C CNN "Part Number"
@@
 F 0 "R16" V 7200 4250 50  0000 C CNN
 F 1 "47R" V 7250 4050 50  0000 C CNN
-F 2 "" V 7180 4050 50  0001 C CNN
+F 2 "Resistors_SMD:R_0603" V 7180 4050 50  0001 C CNN
 F 3 "~" H 7250 4050 50  0001 C CNN
 F 4 "MCWF06P47R0FTL" H 7250 4050 50  0001 C CNN "Part Number"
@@
 F 0 "R9" V 6700 4150 50  0000 C CNN
 F 1 "390R" V 6750 3950 50  0000 C CNN
-F 2 "" V 6680 3950 50  0001 C CNN
+F 2 "Resistors_SMD:R_0603" V 6680 3950 50  0001 C CNN
 F 3 "~" H 6750 3950 50  0001 C CNN
 F 4 "MCWR06X3900FTL" H 6750 3950 50  0001 C CNN "Part Number"
@@
 F 0 "R15" V 7200 4150 50  0000 C CNN
 F 1 "180R" V 7250 3950 50  0000 C CNN
-F 2 "" V 7180 3950 50  0001 C CNN
+F 2 "Resistors_SMD:R_0603" V 7180 3950 50  0001 C CNN
 F 3 "~" H 7250 3950 50  0001 C CNN
 F 4 "MCWR06X1800FTL" H 7250 3950 50  0001 C CNN "Part Number"
@@
 F 0 "R6" V 6700 3850 50  0000 C CNN
 F 1 "2k7" V 6750 3650 50  0000 C CNN
-F 2 "" V 6680 3650 50  0001 C CNN
+F 2 "Resistors_SMD:R_0603" V 6680 3650 50  0001 C CNN
 F 3 "~" H 6750 3650 50  0001 C CNN
 F 4 "MCWR06X2701FTL" H 6750 3650 50  0001 C CNN "Part Number"
@@
 F 0 "R13" V 7200 3950 50  0000 C CNN
 F 1 "820R" V 7250 3750 50  0000 C CNN
-F 2 "" V 7180 3750 50  0001 C CNN
+F 2 "Resistors_SMD:R_0603" V 7180 3750 50  0001 C CNN
 F 3 "~" H 7250 3750 50  0001 C CNN
 F 4 "MCWR06X8200FTL" H 7250 3750 50  0001 C CNN "Part Number"
@@
 F 0 "R8" V 6700 4050 50  0000 C CNN
 F 1 "820R" V 6750 3850 50  0000 C CNN
-F 2 "" V 6680 3850 50  0001 C CNN
+F 2 "Resistors_SMD:R_0603" V 6680 3850 50  0001 C CNN
 F 3 "~" H 6750 3850 50  0001 C CNN
 F 4 "MCWR06X8200FTL" H 6750 3850 50  0001 C CNN "Part Number"
@@
 F 0 "R7" V 6700 3950 50  0000 C CNN
 F 1 "820R" V 6750 3750 50  0000 C CNN
-F 2 "" V 6680 3750 50  0001 C CNN
+F 2 "Resistors_SMD:R_0603" V 6680 3750 50  0001 C CNN
 F 3 "~" H 6750 3750 50  0001 C CNN
 F 4 "MCWR06X8200FTL" H 6750 3750 50  0001 C CNN "Part Number"
@@
 F 0 "R12" V 7200 3850 50  0000 C CNN
 F 1 "220R" V 7250 3650 50  0000 C CNN
-F 2 "" V 7180 3650 50  0001 C CNN
+F 2 "Resistors_SMD:R_0603" V 7180 3650 50  0001 C CNN
 F 3 "~" H 7250 3650 50  0001 C CNN
 F 4 "MCWR06X2200FTL" H 7250 3650 50  0001 C CNN "Part Number"
@@
 F 0 "R5" V 6700 3750 50  0000 C CNN
 F 1 "6k8" V 6750 3550 50  0000 C CNN
-F 2 "" V 6680 3550 50  0001 C CNN
+F 2 "Resistors_SMD:R_0603" V 6680 3550 50  0001 C CNN
 F 3 "~" H 6750 3550 50  0001 C CNN
 F 4 "MCWR06X6801FTL" H 6750 3550 50  0001 C CNN "Part Number"
@@
 F 0 "R11" V 7200 3750 50  0000 C CNN
 F 1 "100R" V 7250 3550 50  0000 C CNN
-F 2 "" V 7180 3550 50  0001 C CNN
+F 2 "Resistors_SMD:R_0603" V 7180 3550 50  0001 C CNN
 F 3 "~" H 7250 3550 50  0001 C CNN
 F 4 "MCWR06X1000FTL" H 7250 3550 50  0001 C CNN "Part Number"
@@
 F 0 "R1" H 2900 2000 50  0000 L CNN
 F 1 "27k" H 2900 1900 50  0000 L CNN
-F 2 "" V 2730 1950 50  0001 C CNN
+F 2 "Resistors_SMD:R_0603" V 2730 1950 50  0001 C CNN
 F 3 "~" H 2800 1950 50  0001 C CNN
 F 4 "MCWR06X2702FTL" H 2800 1950 50  0001 C CNN "Part Number"
@@
 F 0 "R2" V 4600 4100 50  0000 C CNN
 F 1 "1k0" V 4650 3900 50  0000 C CNN
-F 2 "" V 4580 3900 50  0001 C CNN
+F 2 "Resistors_SMD:R_0603" V 4580 3900 50  0001 C CNN
 F 3 "~" H 4650 3900 50  0001 C CNN
 F 4 "MCSR06X1001FTL" H 4650 3900 50  0001 C CNN "Part Number"
@@
 F 0 "J2" H 2680 4292 50  0000 L CNN
 F 1 "2way Screw Terminal" H 2680 4201 50  0000 L CNN
-F 2 "" H 2600 4300 50  0001 C CNN
+F 2 "Terminal_Blocks:TerminalBlock_bornier-2_P5.08mm" H 2600 4300 50  0001 C CNN
 F 3 "~" H 2600 4300 50  0001 C CNN
 F 4 "CTB0102/2" H 2600 4300 50  0001 C CNN "Part Number"

Commit message: Laid out PCB components
Parts:
- D1: footprint Package_TO_SOT_SMD:SOT-23 -> TO_SOT_Packages_SMD:SOT-23
- DC1: footprint (none) -> jakub:XPPOWER_LDU24
- JP1: footprint (none) -> Pin_Headers:Pin_Header_Straight_1x03_Pitch2.54mm
- SW1: footprint (none) -> jakub:switchDPDT
- SW2: footprint (none) -> jakub:Nidec_Copal_SS-10-16
Changed lines of the file:
@@
 F 0 "SW2" V 5654 4937 50  0000 L CNN
 F 1 "6pos rotary" V 5745 4937 50  0000 L CNN
-F 2 "" H 5600 4750 50  0001 C CNN
+F 2 "jakub:Nidec_Copal_SS-10-16" H 5600 4750 50  0001 C CNN
 F 3 "http://www.farnell.com/datasheets/2604296.pdf" H 5600 4750 50  0001 C CNN
 F 4 "SS-10-16NP-LE" H 5700 4150 50  0001 C CNN "Part Number"
-F 5 "Farnell" H 5700 4150 50  0001 C CNN "Distributor"
-F 6 "Nidec Copal" H 5700 4150 50  0001 C CNN "Manufacturer"
-F 7 "2854809" H 5700 4150 50  0001 C CNN "Order Code"
+F 5 "Nidec Copal" H 5700 4150 50  0001 C CNN "Manufacturer"
+F 6 "2854809" H 5700 4150 50  0001 C CNN "Order Code"
+F 7 "Farnell" H 5700 4150 50  0001 C CNN "Distributor"
 F 8 "6-position rotary switch" H 5700 4150 50  0001 C CNN "Description"
 	1    5700 4150
@@
 F 0 "SW1" H 2500 1785 50  0000 C CNN
 F 1 "DPDT Switch" H 2500 1694 50  0000 C CNN
-F 2 "" H 2500 1500 50  0001 C CNN
+F 2 "jakub:switchDPDT" H 2500 1500 50  0001 C CNN
 F 3 "" H 2500 1500 50  0001 C CNN
 F 4 "1MD4T1B1M1QE" H 2500 1500 50  0001 C CNN "Part Number"
@@
 F 0 "SW1" H 7850 1785 50  0000 C CNN
 F 1 "DPDT Switch" H 7850 1694 50  0000 C CNN
-F 2 "" H 7850 1500 50  0001 C CNN
+F 2 "jakub:switchDPDT" H 7850 1500 50  0001 C CNN
 F 3 "" H 7850 1500 50  0001 C CNN
 	2    7850 1500
@@
 F 0 "D1" V 2846 2863 50  0000 R CNN
 F 1 "MAX6006" V 2755 2863 50  0000 R CNN
-F 2 "Package_TO_SOT_SMD:SOT-23" H 2800 2750 50  0001 C CIN
+F 2 "TO_SOT_Packages_SMD:SOT-23" H 2800 2750 50  0001 C CIN
 F 3 "" H 2800 2950 50  0001 C CIN
 F 4 "MAX6006BEUR+T" H 2800 2950 50  0001 C CNN "Part Number"
@@
 F 0 "DC1" H 5900 2267 50  0000 C CNN
 F 1 "LED driver 24V/1A" H 5900 2176 50  0000 C CNN
-F 2 "" H 6100 1450 50  0001 C CNN
+F 2 "jakub:XPPOWER_LDU24" H 6100 1450 50  0001 C CNN
 F 3 "" H 6100 1300 50  0001 C CNN
 F 4 "LDU2430S1000" H 5900 1800 50  0001 C CNN "Part Number"
-F 5 "Farnell" H 5900 1800 50  0001 C CNN "Distributor"
-F 6 "XP Power" H 5900 1800 50  0001 C CNN "Manufacturer"
-F 7 "1738296" H 5900 1800 50  0001 C CNN "Order Code"
+F 5 "XP Power" H 5900 1800 50  0001 C CNN "Manufacturer"
+F 6 "1738296" H 5900 1800 50  0001 C CNN "Order Code"
+F 7 "Farnell" H 5900 1800 50  0001 C CNN "Distributor"
 F 8 "24V/1A adjustable LED driver" H 5900 1800 50  0001 C CNN "Description"
 	1    5900 1800
@@
 F 0 "JP1" V 3804 3966 50  0000 L CNN
 F 1 "Jumper_3_Bridged12" V 3895 3966 50  0000 L CNN
-F 2 "" H 3850 3900 50  0001 C CNN
+F 2 "Pin_Headers:Pin_Header_Straight_1x03_Pitch2.54mm" H 3850 3900 50  0001 C CNN
 F 3 "~" H 3850 3900 50  0001 C CNN
 	1    3850 3900

Commit message: Laid out the PCB
Parts:
- added F1: T1.25A, Fuse_Holders_and_Fuses:Fuseholder5x20_horiz_open_lateral_Type-II, symbol Device:Fuse
- added H1, H2, H3, H4: ⌀3.2mm, Mounting_Holes:MountingHole_3.2mm_M3, symbol Mechanical:MountingHole
- DC1: value LED driver 24V/1A -> LDU2430S1000
- SW2: symbol LEDregulator-rescue:SW_Rotary1x6-jakub -> jakub:SW_Rotary1x6
Connections:
- wire segments 84 -> 85
Other:
- note added: "LED driver 24V/1A"
- note added: "Mounting\nHoles"
- moved on the sheet: C1, C2, C3, C4, D1, DC1, J1, J2, J3, JP1, R1, R10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

Commit message: Board ready
Parts:
- added R5: 120R, Resistors_SMD:R_0603, symbol Device:R
- J2, J3: Description 2way 5mm screw terminal -> 2way 5.08mm screw terminal; Manufacturer CamdenBoss -> Multicomp; Order Code 2493614 -> 2008004; Part Number CTB0102/2 -> MC000034
- R3, R4: value 150R -> 120R; Description 150Ω 0603 1% SMD resistor -> 120Ω 0603 1% SMD resistor; Order Code 2447255 -> 2447240
- renumbered R9 to R10, R10 to R11, R11 to R12, R12 to R13, R13 to R14, R14 to R15, R15 to R16, R16 to R17, R5 to R6, R6 to R7, R7 to R8, R8 to R9
Connections:
- net TrickleOut: now also R5.1; no longer R4.1
- new net: R4.1, R5.2
Changed lines of the file:
@@
 EESchema Schematic File Version 4
 LIBS:LEDregulator-cache
-EELAYER 26 0
+EELAYER 29 0
 EELAYER END
 $Descr A4 11693 8268
@@
 Sheet 1 1
 Title "LED power regulator"
-Date "2019-05-21"
+Date "2019-06-07"
 Rev "0"
 Comp "King's College London"
@@
 Wire Wire Line
 	6900 1600 7000 1600
-$Comp
-L Device:R R3
-U 1 1 5CE564E5
-P 5950 1100
-F 0 "R3" V 5850 1100 50  0000 C CNN
-F 1 "150R" V 5950 1100 50  0000 C CNN
-F 2 "Resistors_SMD:R_0603" V 5880 1100 50  0001 C CNN
-F 3 "~" H 5950 1100 50  0001 C CNN
-F 4 "MCWR06X1500FTL" H 5950 1100 50  0001 C CNN "Part Number"
-F 5 "Farnell" H 5950 1100 50  0001 C CNN "Distributor"
-F 6 "Multicomp" H 5950 1100 50  0001 C CNN "Manufacturer"
-F 7 "2447255" H 5950 1100 50  0001 C CNN "Order Code"
-F 8 "150Ω 0603 1% SMD resistor" H 5950 1100 50  0001 C CNN "Description"
-	1    5950 1100
-	0    1    1    0
-$EndComp
 Wire Wire Line
 	3100 1400 3000 1400
@@
 	6900 3950 6500 3950
 $Comp
-L Device:R R10
+L Device:R R11
 U 1 1 5CE76725
 P 7050 4050
-F 0 "R10" V 7100 4250 50  0000 C CNN
+F 0 "R11" V 7100 4250 50  0000 C CNN
 F 1 "270R" V 7050 4050 50  0000 C CNN
 F 2 "Resistors_SMD:R_0603" V 6980 4050 50  0001 C CNN
@@
 Wire Wire Line
 	7200 4050 7400 4050
-$Comp
-L Connector:Screw_Terminal_01x02 J3
-U 1 1 5CE93AA6
-P 9050 1500
-F 0 "J3" H 9130 1492 50  0000 L CNN
-F 1 "2way Screw Terminal" H 9130 1401 50  0000 L CNN
-F 2 "Terminal_Blocks:TerminalBlock_bornier-2_P5.08mm" H 9050 1500 50  0001 C CNN
-F 3 "~" H 9050 1500 50  0001 C CNN
-F 4 "CTB0102/2" H 9050 1500 50  0001 C CNN "Part Number"
-F 5 "Farnell" H 9050 1500 50  0001 C CNN "Distributor"
-F 6 "CamdenBoss" H 9050 1500 50  0001 C CNN "Manufacturer"
-F 7 "2493614" H 9050 1500 50  0001 C CNN "Order Code"
-F 8 "2way 5mm screw terminal" H 9050 1500 50  0001 C CNN "Description"
-	1    9050 1500
-	1    0    0    -1
-$EndComp
 Wire Wire Line
 	8850 1500 8350 1500
@@
 	5200 4000 5200 3900
 Wire Wire Line
-	6600 1100 7000 1100
-Wire Wire Line
-	6100 1100 6300 1100
-Wire Wire Line
-	5800 1100 3100 1100
+	5900 1100 6000 1100
+Wire Wire Line
+	5600 1100 3100 1100
 $Comp
 L LEDregulator-rescue:LDU2430S1000-jakub DC1
@@
 $EndComp
 $Comp
-L Device:R R4
-U 1 1 5CEAD5AE
-P 6450 1100
-F 0 "R4" V 6350 1100 50  0000 C CNN
-F 1 "150R" V 6450 1100 50  0000 C CNN
-F 2 "Resistors_SMD:R_0603" V 6380 1100 50  0001 C CNN
-F 3 "~" H 6450 1100 50  0001 C CNN
-F 4 "MCWR06X1500FTL" H 6450 1100 50  0001 C CNN "Part Number"
-F 5 "Farnell" H 6450 1100 50  0001 C CNN "Distributor"
-F 6 "Multicomp" H 6450 1100 50  0001 C CNN "Manufacturer"
-F 7 "2447255" H 6450 1100 50  0001 C CNN "Order Code"
-F 8 "150Ω 0603 1% SMD resistor" H 6450 1100 50  0001 C CNN "Description"
-	1    6450 1100
-	0    1    1    0
-$EndComp
-$Comp
-L Device:R R14
+L Device:R R15
 U 1 1 5CEADEEE
 P 7550 3850
-F 0 "R14" V 7500 4050 50  0000 C CNN
+F 0 "R15" V 7500 4050 50  0000 C CNN
 F 1 "150R" V 7550 3850 50  0000 C CNN
 F 2 "Resistors_SMD:R_0603" V 7480 3850 50  0001 C CNN
@@
 $EndComp
 $Comp
-L Device:R R16
+L Device:R R17
 U 1 1 5CEB2542
 P 7550 4050
-F 0 "R16" V 7500 4250 50  0000 C CNN
+F 0 "R17" V 7500 4250 50  0000 C CNN
 F 1 "47R" V 7550 4050 50  0000 C CNN
 F 2 "Resistors_SMD:R_0603" V 7480 4050 50  0001 C CNN
@@
 $EndComp
 $Comp
-L Device:R R9
+L Device:R R10
 U 1 1 5CEB591C
 P 7050 3950
-F 0 "R9" V 7000 4150 50  0000 C CNN
+F 0 "R10" V 7000 4150 50  0000 C CNN
 F 1 "390R" V 7050 3950 50  0000 C CNN
 F 2 "Resistors_SMD:R_0603" V 6980 3950 50  0001 C CNN
@@
 $EndComp
 $Comp
-L Device:R R15
+L Device:R R16
 U 1 1 5CEC2595
 P 7550 3950
-F 0 "R15" V 7500 4150 50  0000 C CNN
+F 0 "R16" V 7500 4150 50  0000 C CNN
 F 1 "180R" V 7550 3950 50  0000 C CNN
 F 2 "Resistors_SMD:R_0603" V 7480 3950 50  0001 C CNN
@@
 $EndComp
 $Comp
-L Device:R R6
+L Device:R R7
 U 1 1 5CECA4F8
 P 7050 3650
-F 0 "R6" V 7000 3850 50  0000 C CNN
+F 0 "R7" V 7000 3850 50  0000 C CNN
 F 1 "2k7" V 7050 3650 50  0000 C CNN
 F 2 "Resistors_SMD:R_0603" V 6980 3650 50  0001 C CNN
@@
 $EndComp
 $Comp
-L Device:R R13
+L Device:R R14
 U 1 1 5CECB7A6
 P 7550 3750
-F 0 "R13" V 7500 3950 50  0000 C CNN
+F 0 "R14" V 7500 3950 50  0000 C CNN
 F 1 "820R" V 7550 3750 50  0000 C CNN
 F 2 "Resistors_SMD:R_0603" V 7480 3750 50  0001 C CNN
@@
 $EndComp
 $Comp
-L Device:R R8
+L Device:R R9
 U 1 1 5CECBAFC
 P 7050 3850
-F 0 "R8" V 7000 4050 50  0000 C CNN
+F 0 "R9" V 7000 4050 50  0000 C CNN
 F 1 "820R" V 7050 3850 50  0000 C CNN
 F 2 "Resistors_SMD:R_0603" V 6980 3850 50  0001 C CNN
@@
 $EndComp
 $Comp
-L Device:R R7
+L Device:R R8
 U 1 1 5CECBF11
 P 7050 3750
-F 0 "R7" V 7000 3950 50  0000 C CNN
+F 0 "R8" V 7000 3950 50  0000 C CNN
 F 1 "820R" V 7050 3750 50  0000 C CNN
 F 2 "Resistors_SMD:R_0603" V 6980 3750 50  0001 C CNN
@@
 $EndComp
 $Comp
-L Device:R R12
+L Device:R R13
 U 1 1 5CECD51D
 P 7550 3650
-F 0 "R12" V 7500 3850 50  0000 C CNN
+F 0 "R13" V 7500 3850 50  0000 C CNN
 F 1 "220R" V 7550 3650 50  0000 C CNN
 F 2 "Resistors_SMD:R_0603" V 7480 3650 50  0001 C CNN
@@
 $EndComp
 $Comp
-L Device:R R5
+L Device:R R6
 U 1 1 5CED022F
 P 7050 3550
-F 0 "R5" V 7000 3750 50  0000 C CNN
+F 0 "R6" V 7000 3750 50  0000 C CNN
 F 1 "6k8" V 7050 3550 50  0000 C CNN
 F 2 "Resistors_SMD:R_0603" V 6980 3550 50  0001 C CNN
@@
 $EndComp
 $Comp
-L Device:R R11
+L Device:R R12
 U 1 1 5CED37E9
 P 7550 3550
-F 0 "R11" V 7500 3750 50  0000 C CNN
+F 0 "R12" V 7500 3750 50  0000 C CNN
 F 1 "100R" V 7550 3550 50  0000 C CNN
 F 2 "Resistors_SMD:R_0603" V 7480 3550 50  0001 C CNN
@@
 F 2 "Terminal_Blocks:TerminalBlock_bornier-2_P5.08mm" H 2900 4300 50  0001 C CNN
 F 3 "~" H 2900 4300 50  0001 C CNN
-F 4 "CTB0102/2" H 2900 4300 50  0001 C CNN "Part Number"
+F 4 "MC000034" H 2900 4300 50  0001 C CNN "Part Number"
 F 5 "Farnell" H 2900 4300 50  0001 C CNN "Distributor"
-F 6 "CamdenBoss" H 2900 4300 50  0001 C CNN "Manufacturer"
-F 7 "2493614" H 2900 4300 50  0001 C CNN "Order Code"
-F 8 "2way 5mm screw terminal" H 2900 4300 50  0001 C CNN "Description"
+F 6 "Multicomp" H 2900 4300 50  0001 C CNN "Manufacturer"
+F 7 "2008004" H 2900 4300 50  0001 C CNN "Order Code"
+F 8 "2way 5.08mm screw terminal" H 2900 4300 50  0001 C CNN "Description"
 	1    2900 4300
 	-1   0    0    -1
@@
 Text Notes 5850 2400 0    50   ~ 0
 LED driver 24V/1A
+$Comp
+L Device:R R5
+U 1 1 5CF9AA93
+P 6550 1100
+F 0 "R5" V 6450 1100 50  0000 C CNN
+F 1 "120R" V 6550 1100 50  0000 C CNN
+F 2 "Resistors_SMD:R_0603" V 6480 1100 50  0001 C CNN
+F 3 "~" H 6550 1100 50  0001 C CNN
+F 4 "MCWR06X1500FTL" H 6550 1100 50  0001 C CNN "Part Number"
+F 5 "Farnell" H 6550 1100 50  0001 C CNN "Distributor"
+F 6 "Multicomp" H 6550 1100 50  0001 C CNN "Manufacturer"
+F 7 "2447240" H 6550 1100 50  0001 C CNN "Order Code"
+F 8 "120Ω 0603 1% SMD resistor" H 6550 1100 50  0001 C CNN "Description"
+	1    6550 1100
+	0    1    1    0
+$EndComp
+Wire Wire Line
+	6400 1100 6300 1100
+Wire Wire Line
+	6700 1100 7000 1100
+$Comp
+L Device:R R4
+U 1 1 5CFA2193
+P 6150 1100
+F 0 "R4" V 6050 1100 50  0000 C CNN
+F 1 "120R" V 6150 1100 50  0000 C CNN
+F 2 "Resistors_SMD:R_0603" V 6080 1100 50  0001 C CNN
+F 3 "~" H 6150 1100 50  0001 C CNN
+F 4 "MCWR06X1500FTL" H 6150 1100 50  0001 C CNN "Part Number"
+F 5 "Farnell" H 6150 1100 50  0001 C CNN "Distributor"
+F 6 "Multicomp" H 6150 1100 50  0001 C CNN "Manufacturer"
+F 7 "2447240" H 6150 1100 50  0001 C CNN "Order Code"
+F 8 "120Ω 0603 1% SMD resistor" H 6150 1100 50  0001 C CNN "Description"
+	1    6150 1100
+	0    1    1    0
+$EndComp
+$Comp
+L Device:R R3
+U 1 1 5CFA27C4
+P 5750 1100
+F 0 "R3" V 5650 1100 50  0000 C CNN
+F 1 "120R" V 5750 1100 50  0000 C CNN
+F 2 "Resistors_SMD:R_0603" V 5680 1100 50  0001 C CNN
+F 3 "~" H 5750 1100 50  0001 C CNN
+F 4 "MCWR06X1500FTL" H 5750 1100 50  0001 C CNN "Part Number"
+F 5 "Farnell" H 5750 1100 50  0001 C CNN "Distributor"
+F 6 "Multicomp" H 5750 1100 50  0001 C CNN "Manufacturer"
+F 7 "2447240" H 5750 1100 50  0001 C CNN "Order Code"
+F 8 "120Ω 0603 1% SMD resistor" H 5750 1100 50  0001 C CNN "Description"
+	1    5750 1100
+	0    1    1    0
+$EndComp
+$Comp
+L Connector:Screw_Terminal_01x02 J3
+U 1 1 5CE93AA6
+P 9050 1500
+F 0 "J3" H 9130 1492 50  0000 L CNN
+F 1 "2way Screw Terminal" H 9130 1401 50  0000 L CNN
+F 2 "Terminal_Blocks:TerminalBlock_bornier-2_P5.08mm" H 9050 1500 50  0001 C CNN
+F 3 "~" H 9050 1500 50  0001 C CNN
+F 4 "MC000034" H 9050 1500 50  0001 C CNN "Part Number"
+F 5 "Farnell" H 9050 1500 50  0001 C CNN "Distributor"
+F 6 "Multicomp" H 9050 1500 50  0001 C CNN "Manufacturer"
+F 7 "2008004" H 9050 1500 50  0001 C CNN "Order Code"
+F 8 "2way 5.08mm screw terminal" H 9050 1500 50  0001 C CNN "Description"
+	1    9050 1500
+	1    0    0    -1
+$EndComp
 $EndSCHEMATC

Commit message: Updated several part details with alternative suppliers
Parts:
- C2: Description 47µF/63V ceramic capacitor D8mm x H10.2mm -> 47µF/63V electrolytic capacitor D8mm x H10.2mm
- JP1: Manufacturer (none) -> Multicomp; Note (none) -> 3way 2.54mm header; Order Code (none) -> 1593412; Package (none) -> 1x3 row; Part Number (none) -> 2211S-03G; Supplier (none) -> Farnell
- R2: Order Code 2074166 -> 2447272; Part Number MCSR06X1001FTL -> MCWR06X1001FTL
Changed lines of the file:
@@
 F 6 "Panasonic" H 4300 1950 50  0001 C CNN "Manufacturer"
 F 7 "2326166" H 4300 1950 50  0001 C CNN "Order Code"
-F 8 "47µF/63V ceramic capacitor D8mm x H10.2mm" H 4300 1950 50  0001 C CNN "Description"
+F 8 "47µF/63V electrolytic capacitor D8mm x H10.2mm" H 4300 1950 50  0001 C CNN "Description"
 	1    4300 1950
 	1    0    0    -1
@@
 F 2 "Resistors_SMD:R_0603" V 4880 3900 50  0001 C CNN
 F 3 "~" H 4950 3900 50  0001 C CNN
-F 4 "MCSR06X1001FTL" H 4950 3900 50  0001 C CNN "Part Number"
+F 4 "MCWR06X1001FTL" H 4950 3900 50  0001 C CNN "Part Number"
 F 5 "Farnell" H 4950 3900 50  0001 C CNN "Distributor"
 F 6 "Multicomp" H 4950 3900 50  0001 C CNN "Manufacturer"
-F 7 "2074166" H 4950 3900 50  0001 C CNN "Order Code"
+F 7 "2447272" H 4950 3900 50  0001 C CNN "Order Code"
 F 8 "1kΩ 0603 1% SMD resistor" H 4950 3900 50  0001 C CNN "Description"
 	1    4950 3900
@@
 F 2 "Pin_Headers:Pin_Header_Straight_1x03_Pitch2.54mm" H 4150 3900 50  0001 C CNN
 F 3 "~" H 4150 3900 50  0001 C CNN
+F 4 "2211S-03G" H 4150 3900 50  0001 C CNN "Part Number"
+F 5 "Multicomp" H 4150 3900 50  0001 C CNN "Manufacturer"
+F 6 "1x3 row" H 4150 3900 50  0001 C CNN "Package"
+F 7 "Farnell" H 4150 3900 50  0001 C CNN "Supplier"
+F 8 "1593412" H 4150 3900 50  0001 C CNN "Order Code"
+F 9 "3way 2.54mm header" H 4150 3900 50  0001 C CNN "Note"
 	1    4150 3900
 	0    -1   1    0

Commit message: Final commit after using on a new computer before a v1.1 branch is created
Parts:
- DC1: symbol LEDregulator-rescue:LDU2430S1000-jakub -> jakub:LDU2430S1000
Changed lines of the file:
@@
 EESchema Schematic File Version 4
 LIBS:LEDregulator-cache
-EELAYER 29 0
+EELAYER 30 0
 EELAYER END
 $Descr A4 11693 8268
@@
 	5600 1100 3100 1100
 $Comp
-L LEDregulator-rescue:LDU2430S1000-jakub DC1
+L jakub:LDU2430S1000 DC1
 U 1 1 5CE70B4D
 P 6200 1800
